Commit message: - so changes to accomodate for the mbzirc needs

File: rotors_description/urdf/ardrone.xacro (robot description, xacro)
@@ -1,6 +1,6 @@
 <?xml version="1.0"?>
-<robot name="ardrone" xmlns:xacro="http://ros.org/wiki/xacro">
+<robot name="$(arg name)" xmlns:xacro="http://ros.org/wiki/xacro">
   <!-- Properties -->
-  <xacro:property name="namespace" value="ardrone" />
+  <xacro:property name="namespace" value="$(arg name)" />
   <xacro:property name="rotor_velocity_slowdown_sim" value="10" />
   <xacro:property name="mesh_file" value="ardrone.dae" />

File: rotors_description/urdf/ardrone_base.xacro (robot description, xacro)
@@ -1,4 +1,4 @@
 <?xml version="1.0"?>
-<robot name="ardrone" xmlns:xacro="http://ros.org/wiki/xacro">
+<robot name="$(arg name)" xmlns:xacro="http://ros.org/wiki/xacro">
   <xacro:include filename="$(find rotors_description)/urdf/component_snippets.xacro" />
   <!-- Instantiate ardrone "mechanics" -->

File: rotors_description/urdf/component_snippets.xacro (robot description, xacro)
@@ -659,7 +659,9 @@
     <link name="${namespace}/hokuyo_laser_link">
       <inertial>
-        <mass value="0.001" />
-        <origin xyz="0 0 0" rpy="0 0 0" />
-        <inertia ixx="0.0001" ixy="0" ixz="0" iyy="0.000001" iyz="0" izz="0.0001" />
+        <mass value="0.00001" />
+        <origin xyz="0 0 0" rpy="0 0 0" />
+        <inertia ixx="0.0000" ixy="0" ixz="0" iyy="0.000000" iyz="0" izz="0.0000" />
+        <!--origin xyz="0 0 0" rpy="0 0 0" />
+        <inertia ixx="0.0001" ixy="0" ixz="0" iyy="0.000001" iyz="0" izz="0.0001" /-->
       </inertial>
       <visual>
@@ -706,7 +708,9 @@
       </ray>
       <plugin name="gazebo_ros_hokuyo_laser" filename="libgazebo_ros_laser.so">
-        <robotNamespace>${namespace}</robotNamespace>
-        <topicName>${namespace}/laser/scan</topicName>
-        <frameName>${namespace}/hokuyo_laser_link</frameName>
+        <gaussianNoise>0.005</gaussianNoise>
+        <alwaysOn>true</alwaysOn>
+        <!--robotNamespace>${namespace}</robotNamespace-->
+        <topicName>scan</topicName>
+        <frameName>hokuyo_laser_link</frameName>
       </plugin>
     </sensor>
