Commit message: - Additions and modifications on iris model and world for aircraft inspection scenario

File: rotors_description/urdf/component_snippets.xacro (robot description, xacro)
@@ -637,3 +637,186 @@
     </xacro:imu_plugin_macro>
   </xacro:macro>
+  <!-- Adding KINECT CAMERA -->
+    <!-- Xacro properties -->
+ <!-- <xacro:property name="M_SCALE" value="0.001"/>-->
+ <!-- <xacro:property name="asus_xtion_pro_offset_cam_py" value="-0.0125"/>-->
+  <xacro:property name="asus_xtion_pro_offset_depth_rel_rgb_py" value="0.0270" />
+  <xacro:property name="asus_xtion_pro_offset_cam_rel_rgb_py"   value="-0.0220" />
+  <!-- Parameterised in part by the values in turtlebot_properties.urdf.xacro -->
+  <xacro:macro name="sensor_asus_xtion_macro" params="namespace parent_link enable_ground_truth *origin">
+    <joint name="${namespace}_camera_rgb_joint" type="fixed">
+      <xacro:insert_block name="origin" />
+      <parent link="${parent_link}"/>
+      <child link="${namespace}/camera_rgb_frame" />
+    </joint>
+    <link name="${namespace}/camera_rgb_frame"/>
+    <joint name="${namespace}_camera_rgb_optical_joint" type="fixed">
+      <origin xyz="0 0 0" rpy="${-pi/2} 0 ${-pi/2}" />
+      <parent link="${namespace}/camera_rgb_frame" />
+      <child link="${namespace}/camera_rgb_optical_frame" />
+    </joint>
+    <link name="${namespace}/camera_rgb_optical_frame"/>
+    <joint name="${namespace}_camera_joint" type="fixed">
+      <origin xyz="0 ${asus_xtion_pro_offset_cam_rel_rgb_py} 0"
+              rpy="0 0 0"/>
+      <parent link="${namespace}/camera_rgb_frame"/>
+      <child link="${namespace}/camera_link"/>
+    </joint>
+    <link name="${namespace}/camera_link">
+      <visual>
+        <origin xyz="-0.015 0.0035 0.004" rpy="${-pi/2} -${pi} ${-pi/2}"/>
+        <geometry>
+          <mesh filename="package://rotors_description/meshes/asus_xtion_pro_live.dae" scale="0.001 0.001 0.001"/>
+        </geometry>
+      </visual>
+      <collision>
+        <origin xyz="0.0 0.0 0.0" rpy="0 0 0" />
+        <geometry>
+        <box size="0.0730 0.2760 0.0720"/>
+      </geometry>
+      </collision>
+      <inertial>
+        <mass value="0.170" />
+        <origin xyz="0 0 0" />
+        <inertia ixx="0.001152600" ixy="0.0" ixz="0.0"
+                 iyy="0.000148934" iyz="0.0"
+                 izz="0.001154654" />
+      </inertial>
+    </link>
+    <joint name="${namespace}_camera_depth_joint" type="fixed">
+      <origin xyz="0 ${asus_xtion_pro_offset_depth_rel_rgb_py} 0" rpy="0 0 0" />
+      <parent link="${namespace}/camera_rgb_frame" />
+      <child link="${namespace}/camera_depth_frame" />
+    </joint>
+    <link name="${namespace}/camera_depth_frame"/>
+    <joint name="${namespace}_camera_depth_optical_joint" type="fixed">
+      <origin xyz="0 0 0" rpy="${-pi/2} 0 ${-pi/2}" />
+      <parent link="${namespace}/camera_depth_frame" />
+      <child link="${namespace}/camera_depth_optical_frame" />
+    </joint>
+    <link name="${namespace}/camera_depth_optical_frame"/>
+      <gazebo reference="${namespace}/camera_link">
+      <sensor type="depth" name="${namespace}_camera">
+        <always_on>true</always_on>
+        <update_rate>20.0</update_rate>
+        <camera>
+          <horizontal_fov>${60.0*pi/180.0}</horizontal_fov>
+          <image>
+            <format>R8G8B8</format>
+            <width>640</width>
+            <height>480</height>
+          </image>
+          <clip>
+            <near>0.05</near>
+            <far>8.0</far>
+          </clip>
+        </camera>
+        <plugin name="${namespace}_camera" filename="libgazebo_ros_openni_kinect.so">
+	  <robotNamespace>${namespace}</robotNamespace>
+          <cameraName>${namespace}_camera</cameraName>
+          <alwaysOn>true</alwaysOn>
+          <updateRate>10</updateRate>
+          <imageTopicName>rgb/image_raw</imageTopicName>
+          <depthImageTopicName>depth/image_raw</depthImageTopicName>
+          <pointCloudTopicName>depth/points</pointCloudTopicName>
+          <cameraInfoTopicName>rgb/camera_info</cameraInfoTopicName>
+          <depthImageCameraInfoTopicName>depth/camera_info</depthImageCameraInfoTopicName>
+          <frameName>camera_depth_optical_frame</frameName>
+          <baseline>0.1</baseline>
+          <distortion_k1>0.0</distortion_k1>
+          <distortion_k2>0.0</distortion_k2>
+          <distortion_k3>0.0</distortion_k3>
+          <distortion_t1>0.0</distortion_t1>
+          <distortion_t2>0.0</distortion_t2>
+          <pointCloudCutoff>0.4</pointCloudCutoff>
+        </plugin>
+      </sensor>
+    </gazebo>
+        <!-- Groundtruth -->
+    <xacro:if value="${enable_ground_truth}">
+      <!-- Odometry Sensor -->
+      <xacro:odometry_plugin_macro
+        namespace="${namespace}/ground_truth"
+        odometry_sensor_suffix=""
+        parent_link="${namespace}/camera_link"
+        pose_topic="pose"
+        pose_with_covariance_topic="pose_with_covariance"
+        position_topic="position"
+        transform_topic="transform"
+        odometry_topic="odometry"
+        parent_frame_id="world"
+        mass_odometry_sensor="0.00001"
+        measurement_divisor="1"
+        measurement_delay="0"
+        unknown_delay="0.0"
+        noise_normal_position="0 0 0"
+        noise_normal_quaternion="0 0 0"
+        noise_normal_linear_velocity="0 0 0"
+        noise_normal_angular_velocity="0 0 0"
+        noise_uniform_position="0 0 0"
+        noise_uniform_quaternion="0 0 0"
+        noise_uniform_linear_velocity="0 0 0"
+        noise_uniform_angular_velocity="0 0 0"
+        enable_odometry_map="false"
+        odometry_map=""
+        image_scale="">
+        <inertia ixx="0.00001" ixy="0.0" ixz="0.0" iyy="0.00001" iyz="0.0" izz="0.00001" /> <!-- [kg m^2] [kg m^2] [kg m^2] [kg m^2] [kg m^2] [kg m^2] -->
+        <origin xyz="0.0 0.0 0.0" rpy="0.0 0.0 0.0" />
+      </xacro:odometry_plugin_macro>
+    </xacro:if>
+  </xacro:macro>
+  <!-- trial kinect -->
+<!--   <xacro:macro name="kinect_macro" params="namespace parent_link">
+  <gazebo>
+<include>
+        <uri>model://kinect</uri>
+        <pose>0.005 0 -0.055 0 ${-1*pi} ${-1*pi}</pose>
+      </include>
+      <joint name="centercam" type="revolute">
+        <child>kinect::link</child>
+        <parent>${parent_link}</parent>
+        <axis>
+          <xyz>1 1 1</xyz>
+          <limit>
+            <upper>0</upper>
+            <lower>0</lower>
+          </limit>
+        </axis>
+      </joint>
+      <sensor type="depth" name="kinect_camera">
+        <always_on>true</always_on>
+        <update_rate>20.0</update_rate>
+        <camera>
+          <horizontal_fov>${60.0*pi/180.0}</horizontal_fov>
+          <image>
+            <format>R8G8B8</format>
+            <width>640</width>
+            <height>480</height>
+          </image>
+          <clip>
+            <near>0.05</near>
+            <far>8.0</far>
+          </clip>
+        </camera>
+        <plugin name="kinect_camera" filename="libgazebo_ros_openni_kinect.so">
+          <cameraName>kinect_camera</cameraName>
+          <alwaysOn>true</alwaysOn>
+          <updateRate>10</updateRate>
+          <imageTopicName>rgb/image_raw</imageTopicName>
+          <depthImageTopicName>depth/image_raw</depthImageTopicName>
+          <pointCloudTopicName>depth/points</pointCloudTopicName>
+          <cameraInfoTopicName>rgb/camera_info</cameraInfoTopicName>
+          <depthImageCameraInfoTopicName>depth/camera_info</depthImageCameraInfoTopicName>
+          <frameName>camera_depth_frame</frameName>
+          <baseline>0.1</baseline>
+          <distortion_k1>0.0</distortion_k1>
+          <distortion_k2>0.0</distortion_k2>
+          <distortion_k3>0.0</distortion_k3>
+          <distortion_t1>0.0</distortion_t1>
+          <distortion_t2>0.0</distortion_t2>
+          <pointCloudCutoff>0.4</pointCloudCutoff>
+        </plugin>
+      </sensor>
+</gazebo>
+   </xacro:macro> -->
 </robot>

Commit message: - added laser sensor and a new testing world

File: rotors_description/urdf/component_snippets.xacro (robot description, xacro)
@@ -766,4 +766,67 @@
     </xacro:if>
   </xacro:macro>
+  <!-- Hokuyo LIDAR for simulation -->
+  <xacro:macro name="hokuyo_laser" params="namespace parent_link *origin">
+   <joint name="${namespace}/hokuyo_laser_joint" type="fixed">
+      <axis xyz="0 1 0" />
+      <xacro:insert_block name="origin" />
+      <parent link="${parent_link}"/>
+      <child link="${namespace}/hokuyo_laser_link"/>
+    </joint>
+    <link name="${namespace}/hokuyo_laser_link">
+      <inertial>
+        <mass value="0.001" />
+        <origin xyz="0 0 0" rpy="0 0 0" />
+        <inertia ixx="0.0001" ixy="0" ixz="0" iyy="0.000001" iyz="0" izz="0.0001" />
+      </inertial>
+      <visual>
+        <origin xyz="0 0 0" rpy="0 0 0" />
+        <geometry>
+          <mesh filename="package://rotors_description/meshes/hokuyo.dae"/>
+        </geometry>
+      </visual>
+      <collision>
+	<origin xyz="0 0 0" rpy="0 0 0" />
+	<geometry>
+	  <mesh filename="package://rotors_description/meshes/hokuyo.dae"/>
+	</geometry>
+      </collision>
+    </link>
+  <gazebo reference="${namespace}/hokuyo_laser_link">
+    <sensor type="ray" name="${namespace}/hokuyo_laser">
+      <pose>0 0 0 0 0 0</pose>
+      <visualize>true</visualize>
+      <update_rate>40</update_rate>
+      <ray>
+        <scan>
+          <horizontal>
+            <samples>720</samples>
+            <resolution>1</resolution>
+            <min_angle>-1.570796</min_angle>
+            <max_angle>1.570796</max_angle>
+          </horizontal>
+        </scan>
+        <range>
+          <min>0.10</min>
+          <max>30.0</max>
+          <resolution>0.01</resolution>
+        </range>
+        <noise>
+          <type>gaussian</type>
+          <!-- Noise parameters based on published spec for Hokuyo laser
+               achieving "+-30mm" accuracy at range < 10m.  A mean of 0.0m and
+               stddev of 0.01m will put 99.7% of samples within 0.03m of the true
+               reading. -->
+          <mean>0.0</mean>
+          <stddev>0.01</stddev>
+        </noise>
+      </ray>
+      <plugin name="gazebo_ros_hokuyo_laser" filename="libgazebo_ros_laser.so">
+        <topicName>laser/scan</topicName>
+        <frameName>${namespace}/hokuyo_laser_link</frameName>
+      </plugin>
+    </sensor>
+  </gazebo>
+  </xacro:macro>
   <!-- trial kinect -->
 <!--   <xacro:macro name="kinect_macro" params="namespace parent_link">

Commit message: - added camera sensor , the frame is /iris/camera_sensor/camera_link for Rviz

File: rotors_description/urdf/component_snippets.xacro (robot description, xacro)
@@ -766,4 +766,104 @@
     </xacro:if>
   </xacro:macro>
+<!--  *****************************************************************  -->
+<!-- Adding REgular CAMERA -->
+<xacro:macro name="sensor_camera_macro" params="namespace parent_link enable_ground_truth *origin">
+  <joint name="camera_joint" type="fixed">
+    <axis xyz="0 1 0" />
+    <xacro:insert_block name="origin" />
+    <parent link="${parent_link}"/>
+    <child link="${namespace}/camera_link"/>
+  </joint>
+  <link name="${namespace}/camera_link">
+    <collision>
+      <origin xyz="-0.03 0 0" rpy="0 0 0"/>
+      <geometry>
+<!--    <box size="${camera_link} ${camera_link} ${camera_link}"/>-->
+          <mesh filename="package://rotors_description/meshes/hokuyo.dae"/>
+      </geometry>
+    </collision>
+    <visual>
+      <origin xyz="-0.03 0 0" rpy="0 0 0"/>
+      <geometry>
+<!--     <box size="${camera_link} ${camera_link} ${camera_link}"/> -->
+          <mesh filename="package://rotors_description/meshes/hokuyo.dae"/>
+      </geometry>
+      <material name="red"/>
+    </visual>
+    <inertial>
+      <mass value="1e-5" />
+      <origin xyz="0 0 0" rpy="0 0 0"/>
+      <inertia ixx="1e-6" ixy="0" ixz="0" iyy="1e-6" iyz="0" izz="1e-6" />
+    </inertial>
+  </link>
+  <gazebo reference="${namespace}/camera_link">
+    <sensor type="camera" name="${namespace}_camera1">
+      <update_rate>30.0</update_rate>
+      <camera name="head">
+        <horizontal_fov>1.3962634</horizontal_fov>
+        <image>
+          <width>800</width>
+          <height>800</height>
+          <format>R8G8B8</format>
+        </image>
+        <clip>
+          <near>0.02</near>
+          <far>300</far>
+        </clip>
+        <noise>
+          <type>gaussian</type>
+          <mean>0.0</mean>
+          <stddev>0.007</stddev>
+        </noise>
+      </camera>
+      <plugin name="${namespace}_camera_controller" filename="libgazebo_ros_camera.so">
+	<robotNamespace>${namespace}</robotNamespace>
+        <alwaysOn>true</alwaysOn>
+        <updateRate>10.0</updateRate>
+        <cameraName>${namespace}_camera</cameraName>
+        <imageTopicName>image_raw</imageTopicName>
+        <cameraInfoTopicName>camera_info</cameraInfoTopicName>
+        <frameName>camera_link</frameName>
+        <hackBaseline>0.07</hackBaseline>
+        <distortionK1>0.0</distortionK1>
+        <distortionK2>0.0</distortionK2>
+        <distortionK3>0.0</distortionK3>
+        <distortionT1>0.0</distortionT1>
+        <distortionT2>0.0</distortionT2>
+      </plugin>
+    </sensor>
+  </gazebo>
+    <xacro:if value="${enable_ground_truth}">
+      <xacro:odometry_plugin_macro
+        namespace="${namespace}/ground_truth"
+        odometry_sensor_suffix=""
+        parent_link="${namespace}/camera_link"
+        pose_topic="pose"
+        pose_with_covariance_topic="pose_with_covariance"
+        position_topic="position"
+        transform_topic="transform"
+        odometry_topic="odometry"
+        parent_frame_id="world"
+        mass_odometry_sensor="0.00001"
+        measurement_divisor="1"
+        measurement_delay="0"
+        unknown_delay="0.0"
+        noise_normal_position="0 0 0"
+        noise_normal_quaternion="0 0 0"
+        noise_normal_linear_velocity="0 0 0"
+        noise_normal_angular_velocity="0 0 0"
+        noise_uniform_position="0 0 0"
+        noise_uniform_quaternion="0 0 0"
+        noise_uniform_linear_velocity="0 0 0"
+        noise_uniform_angular_velocity="0 0 0"
+        enable_odometry_map="false"
+        odometry_map=""
+        image_scale="">
+        <inertia ixx="0.00001" ixy="0.0" ixz="0.0" iyy="0.00001" iyz="0.0" izz="0.00001" />
+        <origin xyz="0.0 0.0 0.0" rpy="0.0 0.0 0.0" />
+      </xacro:odometry_plugin_macro>
+    </xacro:if>
+  </xacro:macro>
+<!--  *****************************************************************  -->
   <!-- Hokuyo LIDAR for simulation -->
   <xacro:macro name="hokuyo_laser" params="namespace parent_link *origin">
