Commit message: - added mbzirc model

File: rotors_description/urdf/component_snippets.xacro (robot description, xacro)
@@ -17,5 +17,4 @@
 -->
 <robot xmlns:xacro="http://ros.org/wiki/xacro">
-  <xacro:property name="pi" value="3.14159265359" />
   <!-- Macro to add logging to a bag file. -->
   <xacro:macro name="bag_plugin_macro"
@@ -106,120 +105,4 @@
     </gazebo>
   </xacro:macro>
-  <!-- Camera joint macro - just the joints, links, and collisions for a single
-       camera. -->
-  <xacro:macro name="camera_joint_macro"
-    params="namespace parent_link camera_suffix enable_visual *origin *geometry" >
-    <link name="${namespace}/camera_${camera_suffix}_link">
-      <collision>
-        <origin xyz="0 0 0" rpy="0 0 0" />
-        <geometry>
-          <xacro:insert_block name="geometry" />
-        </geometry>
-      </collision>
-      <xacro:if value="${enable_visual}">
-        <visual>
-          <origin xyz="0 0 0" rpy="0 0 0" />
-          <geometry>
-            <xacro:insert_block name="geometry" />
-          </geometry>
-          <material name="red" />
-        </visual>
-      </xacro:if>
-      <inertial>
-        <mass value="1e-5" />
-        <origin xyz="0 0 0" rpy="0 0 0" />
-        <inertia ixx="1e-6" ixy="0" ixz="0" iyy="1e-6" iyz="0" izz="1e-6" />
-      </inertial>
-    </link>
-    <joint name="${namespace}/camera_${camera_suffix}_joint" type="fixed">
-      <xacro:insert_block name="origin" />
-      <parent link="${parent_link}" />
-      <child link="${namespace}/camera_${camera_suffix}_link" />
-    </joint>
-  </xacro:macro>
-  <!-- Camera sensor macro - just image parameters. -->
-  <xacro:macro name="camera_sensor_macro"
-    params="camera_suffix horizontal_fov image_width image_height
-      image_format min_distance max_distance noise_mean noise_stddev
-      baseline" >
-    <camera name="${camera_suffix}">
-      <pose>0 ${-baseline} 0 0 0 0</pose>
-      <horizontal_fov>${horizontal_fov}</horizontal_fov>
-      <image>
-        <width>${image_width}</width>
-        <height>${image_height}</height>
-        <format>${image_format}</format>
-      </image>
-      <clip>
-        <near>${min_distance}</near>
-        <far>${max_distance}</far>
-      </clip>
-      <noise>
-        <type>gaussian</type>
-        <!-- Noise is sampled independently per pixel on each frame.
-             That pixel's noise value is added to each of its color
-             channels, which at that point lie in the range [0,1]. -->
-        <mean>${noise_mean}</mean>
-        <stddev>${noise_stddev}</stddev>
-      </noise>
-    </camera>
-  </xacro:macro>
-  <!-- Macro to add a multicamera (stereo pair). -->
-  <xacro:macro name="stereo_camera_macro"
-    params="namespace camera_name parent_link frame_rate
-      horizontal_fov image_width image_height image_format min_distance
-      max_distance noise_mean noise_stddev enable_visual origin_offset_x
-      baseline_y origin_offset_z *geometry">
-    <!-- These are parameters for the left camera link and then the right
-        as well. -->
-    <xacro:camera_joint_macro namespace="${namespace}"
-      parent_link="${parent_link}"
-      camera_suffix="left" enable_visual="${enable_visual}">
-      <origin xyz="${origin_offset_x} ${baseline_y/2} ${origin_offset_z}" rpy="0 0 0" />
-      <xacro:insert_block name="geometry" />
-    </xacro:camera_joint_macro>
-    <xacro:camera_joint_macro namespace="${namespace}"
-      parent_link="${parent_link}"
-      camera_suffix="right" enable_visual="${enable_visual}">
-      <origin xyz="${origin_offset_x} ${-baseline_y/2} ${origin_offset_z}" rpy="0 0 0" />
-      <xacro:insert_block name="geometry" />
-    </xacro:camera_joint_macro>
-    <!-- Both cameras in the pair are anchored off the left camera frame. -->
-    <gazebo reference="${namespace}/camera_left_link">
-      <sensor type="multicamera" name="${namespace}_stereo_camera">
-        <update_rate>${frame_rate}</update_rate>
-        <!-- Here we set up the individual cameras of the stereo head. -->
-        <xacro:camera_sensor_macro camera_suffix="left"
-            horizontal_fov="${horizontal_fov}" image_width="${image_width}"
-            image_height="${image_height}" image_format="${image_format}"
-            min_distance="${min_distance}" max_distance="${max_distance}"
-            noise_mean="${noise_mean}" noise_stddev="${noise_stddev}"
-            baseline="0">
-        </xacro:camera_sensor_macro>
-        <xacro:camera_sensor_macro camera_suffix="right"
-            horizontal_fov="${horizontal_fov}" image_width="${image_width}"
-            image_height="${image_height}" image_format="${image_format}"
-            min_distance="${min_distance}" max_distance="${max_distance}"
-            noise_mean="${noise_mean}" noise_stddev="${noise_stddev}"
-            baseline="${baseline_y}">
-        </xacro:camera_sensor_macro>
-        <!-- Stereo controller, setting the transforms between the two cameras. -->
-        <plugin name="${namespace}_stereo_camera_controller" filename="libgazebo_ros_multicamera.so">
-          <alwaysOn>true</alwaysOn>
-          <updateRate>0.0</updateRate>
-          <cameraName>${camera_name}</cameraName>
-          <imageTopicName>image_raw</imageTopicName>
-          <cameraInfoTopicName>camera_info</cameraInfoTopicName>
-          <frameName>${camera_name}/camera_left_link</frameName>
-          <hackBaseline>${baseline_y}</hackBaseline>
-          <distortionK1>0.0</distortionK1>
-          <distortionK2>0.0</distortionK2>
-          <distortionK3>0.0</distortionK3>
-          <distortionT1>0.0</distortionT1>
-          <distortionT2>0.0</distortionT2>
-        </plugin>
-      </sensor>
-    </gazebo>
-  </xacro:macro>
   <!-- Macro to add the controller interface. -->
   <xacro:macro name="controller_plugin_macro" params="namespace imu_sub_topic">
@@ -429,5 +312,5 @@
     <link name="${namespace}/camera_${camera_suffix}_optical_center_link" />
     <joint name="${namespace}/camera_${camera_suffix}_optical_center_joint" type="fixed">
-      <origin xyz="0 0 0" rpy="${-pi/2} 0 ${-pi/2}" />
+      <origin xyz="0 0 0" rpy="${-PI/2} 0 ${-PI/2}" />
       <parent link="${namespace}/camera_${camera_suffix}_link" />
       <child link="${namespace}/camera_${camera_suffix}_optical_center_link" />
@@ -766,104 +649,4 @@
     </xacro:if>
   </xacro:macro>
-<!--  *****************************************************************  -->
-<!-- Adding REgular CAMERA -->
-<xacro:macro name="sensor_camera_macro" params="namespace parent_link enable_ground_truth *origin">
-  <joint name="camera_joint" type="fixed">
-    <axis xyz="0 1 0" />
-    <xacro:insert_block name="origin" />
-    <parent link="${parent_link}"/>
-    <child link="${namespace}/camera_link"/>
-  </joint>
-  <link name="${namespace}/camera_link">
-    <collision>
-      <origin xyz="-0.03 0 0" rpy="0 0 0"/>
-      <geometry>
-<!--    <box size="${camera_link} ${camera_link} ${camera_link}"/>-->
-          <mesh filename="package://rotors_description/meshes/hokuyo.dae"/>
-      </geometry>
-    </collision>
-    <visual>
-      <origin xyz="-0.03 0 0" rpy="0 0 0"/>
-      <geometry>
-<!--     <box size="${camera_link} ${camera_link} ${camera_link}"/> -->
-          <mesh filename="package://rotors_description/meshes/hokuyo.dae"/>
-      </geometry>
-      <material name="red"/>
-    </visual>
-    <inertial>
-      <mass value="1e-5" />
-      <origin xyz="0 0 0" rpy="0 0 0"/>
-      <inertia ixx="1e-6" ixy="0" ixz="0" iyy="1e-6" iyz="0" izz="1e-6" />
-    </inertial>
-  </link>
-  <gazebo reference="${namespace}/camera_link">
-    <sensor type="camera" name="${namespace}_camera1">
-      <update_rate>30.0</update_rate>
-      <camera name="head">
-        <horizontal_fov>1.3962634</horizontal_fov>
-        <image>
-          <width>800</width>
-          <height>800</height>
-          <format>R8G8B8</format>
-        </image>
-        <clip>
-          <near>0.02</near>
-          <far>300</far>
-        </clip>
-        <noise>
-          <type>gaussian</type>
-          <mean>0.0</mean>
-          <stddev>0.007</stddev>
-        </noise>
-      </camera>
-      <plugin name="${namespace}_camera_controller" filename="libgazebo_ros_camera.so">
-	<robotNamespace>${namespace}</robotNamespace>
-        <alwaysOn>true</alwaysOn>
-        <updateRate>10.0</updateRate>
-        <cameraName>${namespace}_camera</cameraName>
-        <imageTopicName>image_raw</imageTopicName>
-        <cameraInfoTopicName>camera_info</cameraInfoTopicName>
-        <frameName>camera_link</frameName>
-        <hackBaseline>0.07</hackBaseline>
-        <distortionK1>0.0</distortionK1>
-        <distortionK2>0.0</distortionK2>
-        <distortionK3>0.0</distortionK3>
-        <distortionT1>0.0</distortionT1>
-        <distortionT2>0.0</distortionT2>
-      </plugin>
-    </sensor>
-  </gazebo>
-    <xacro:if value="${enable_ground_truth}">
-      <xacro:odometry_plugin_macro
-        namespace="${namespace}/ground_truth"
-        odometry_sensor_suffix=""
-        parent_link="${namespace}/camera_link"
-        pose_topic="pose"
-        pose_with_covariance_topic="pose_with_covariance"
-        position_topic="position"
-        transform_topic="transform"
-        odometry_topic="odometry"
-        parent_frame_id="world"
-        mass_odometry_sensor="0.00001"
-        measurement_divisor="1"
-        measurement_delay="0"
-        unknown_delay="0.0"
-        noise_normal_position="0 0 0"
-        noise_normal_quaternion="0 0 0"
-        noise_normal_linear_velocity="0 0 0"
-        noise_normal_angular_velocity="0 0 0"
-        noise_uniform_position="0 0 0"
-        noise_uniform_quaternion="0 0 0"
-        noise_uniform_linear_velocity="0 0 0"
-        noise_uniform_angular_velocity="0 0 0"
-        enable_odometry_map="false"
-        odometry_map=""
-        image_scale="">
-        <inertia ixx="0.00001" ixy="0.0" ixz="0.0" iyy="0.00001" iyz="0.0" izz="0.00001" />
-        <origin xyz="0.0 0.0 0.0" rpy="0.0 0.0 0.0" />
-      </xacro:odometry_plugin_macro>
-    </xacro:if>
-  </xacro:macro>
-<!--  *****************************************************************  -->
   <!-- Hokuyo LIDAR for simulation -->
   <xacro:macro name="hokuyo_laser" params="namespace parent_link *origin">
@@ -929,4 +712,120 @@
     </sensor>
   </gazebo>
+  </xacro:macro>
+    <!-- Camera joint macro - just the joints, links, and collisions for a single
+       camera. -->
+  <xacro:macro name="camera_joint_macro"
+    params="namespace parent_link camera_suffix enable_visual *origin *geometry" >
+    <link name="${namespace}/camera_${camera_suffix}_link">
+      <collision>
+        <origin xyz="0 0 0" rpy="0 0 0" />
+        <geometry>
+          <xacro:insert_block name="geometry" />
+        </geometry>
+      </collision>
+      <xacro:if value="${enable_visual}">
+        <visual>
+          <origin xyz="0 0 0" rpy="0 0 0" />
+          <geometry>
+            <xacro:insert_block name="geometry" />
+          </geometry>
+          <material name="red" />
+        </visual>
+      </xacro:if>
+      <inertial>
+        <mass value="1e-5" />
+        <origin xyz="0 0 0" rpy="0 0 0" />
+        <inertia ixx="1e-6" ixy="0" ixz="0" iyy="1e-6" iyz="0" izz="1e-6" />
+      </inertial>
+    </link>
+    <joint name="${namespace}/camera_${camera_suffix}_joint" type="fixed">
+      <xacro:insert_block name="origin" />
+      <parent link="${parent_link}" />
+      <child link="${namespace}/camera_${camera_suffix}_link" />
+    </joint>
+  </xacro:macro>
+  <!-- Camera sensor macro - just image parameters. -->
+  <xacro:macro name="camera_sensor_macro"
+    params="camera_suffix horizontal_fov image_width image_height
+      image_format min_distance max_distance noise_mean noise_stddev
+      baseline" >
+    <camera name="${camera_suffix}">
+      <pose>0 ${-baseline} 0 0 0 0</pose>
+      <horizontal_fov>${horizontal_fov}</horizontal_fov>
+      <image>
+        <width>${image_width}</width>
+        <height>${image_height}</height>
+        <format>${image_format}</format>
+      </image>
+      <clip>
+        <near>${min_distance}</near>
+        <far>${max_distance}</far>
+      </clip>
+      <noise>
+        <type>gaussian</type>
+        <!-- Noise is sampled independently per pixel on each frame.
+             That pixel's noise value is added to each of its color
+             channels, which at that point lie in the range [0,1]. -->
+        <mean>${noise_mean}</mean>
+        <stddev>${noise_stddev}</stddev>
+      </noise>
+    </camera>
+  </xacro:macro>
+  <!-- Macro to add a multicamera (stereo pair). -->
+  <xacro:macro name="stereo_camera_macro"
+    params="namespace camera_name parent_link frame_rate
+      horizontal_fov image_width image_height image_format min_distance
+      max_distance noise_mean noise_stddev enable_visual origin_offset_x
+      baseline_y origin_offset_z *geometry">
+    <!-- These are parameters for the left camera link and then the right
+        as well. -->
+    <xacro:camera_joint_macro namespace="${namespace}"
+      parent_link="${parent_link}"
+      camera_suffix="left" enable_visual="${enable_visual}">
+      <origin xyz="${origin_offset_x} ${baseline_y/2} ${origin_offset_z}" rpy="0 0 0" />
+      <xacro:insert_block name="geometry" />
+    </xacro:camera_joint_macro>
+    <xacro:camera_joint_macro namespace="${namespace}"
+      parent_link="${parent_link}"
+      camera_suffix="right" enable_visual="${enable_visual}">
+      <origin xyz="${origin_offset_x} ${-baseline_y/2} ${origin_offset_z}" rpy="0 0 0" />
+      <xacro:insert_block name="geometry" />
+    </xacro:camera_joint_macro>
+    <!-- Both cameras in the pair are anchored off the left camera frame. -->
+    <gazebo reference="${namespace}/camera_left_link">
+      <sensor type="multicamera" name="${namespace}_stereo_camera">
+        <update_rate>${frame_rate}</update_rate>
+        <!-- Here we set up the individual cameras of the stereo head. -->
+        <xacro:camera_sensor_macro camera_suffix="left"
+            horizontal_fov="${horizontal_fov}" image_width="${image_width}"
+            image_height="${image_height}" image_format="${image_format}"
+            min_distance="${min_distance}" max_distance="${max_distance}"
+            noise_mean="${noise_mean}" noise_stddev="${noise_stddev}"
+            baseline="0">
+        </xacro:camera_sensor_macro>
+        <xacro:camera_sensor_macro camera_suffix="right"
+            horizontal_fov="${horizontal_fov}" image_width="${image_width}"
+            image_height="${image_height}" image_format="${image_format}"
+            min_distance="${min_distance}" max_distance="${max_distance}"
+            noise_mean="${noise_mean}" noise_stddev="${noise_stddev}"
+            baseline="${baseline_y}">
+        </xacro:camera_sensor_macro>
+        <!-- Stereo controller, setting the transforms between the two cameras. -->
+        <plugin name="${namespace}_stereo_camera_controller" filename="libgazebo_ros_multicamera.so">
+          <alwaysOn>true</alwaysOn>
+          <updateRate>0.0</updateRate>
+          <cameraName>${camera_name}</cameraName>
+          <imageTopicName>image_raw</imageTopicName>
+          <cameraInfoTopicName>camera_info</cameraInfoTopicName>
+          <frameName>${camera_name}/camera_left_link</frameName>
+          <hackBaseline>${baseline_y}</hackBaseline>
+          <distortionK1>0.0</distortionK1>
+          <distortionK2>0.0</distortionK2>
+          <distortionK3>0.0</distortionK3>
+          <distortionT1>0.0</distortionT1>
+          <distortionT2>0.0</distortionT2>
+        </plugin>
+      </sensor>
+    </gazebo>
   </xacro:macro>
   <!-- trial kinect -->

File: rotors_description/urdf/iris.xacro (robot description, xacro)
@@ -35,13 +35,8 @@
   <xacro:property name="rotor_inertia">
     <inertia
-    ixx="9.7500e-07"
-    iyy="1.6670e-04"
-    izz="1.6760e-04"
-    ixy="0.0" ixz="0.0"  iyz="0.0" /> <!-- [kg.m^2] [kg.m^2] [kg.m^2] [kg.m^2] [kg.m^2] [kg.m^2] -->
-    <!--inertia
     ixx="${1/12 * mass_rotor * (0.015 * 0.015 + 0.003 * 0.003) * rotor_velocity_slowdown_sim}"
     iyy="${1/12 * mass_rotor * (4 * radius_rotor * radius_rotor + 0.003 * 0.003) * rotor_velocity_slowdown_sim}"
     izz="${1/12 * mass_rotor * (4 * radius_rotor * radius_rotor + 0.015 * 0.015) * rotor_velocity_slowdown_sim}"
-    ixy="0.0" ixz="0.0"  iyz="0.0" /--> <!-- [kg.m^2] [kg.m^2] [kg.m^2] [kg.m^2] [kg.m^2] [kg.m^2] -->
+    ixy="0.0" ixz="0.0"  iyz="0.0" /> <!-- [kg.m^2] [kg.m^2] [kg.m^2] [kg.m^2] [kg.m^2] [kg.m^2] -->
   </xacro:property>
   <!-- Included URDF Files -->

File: rotors_description/urdf/vi_sensor_base.xacro (robot description, xacro)
@@ -2,5 +2,4 @@
 <robot name="vi_sensor" xmlns:xacro="http://www.ros.org/wiki/xacro">
   <xacro:property name="namespace" value="vi_sensor" />
-  <xacro:property name="PI" value="3.141592654" />
   <xacro:include filename="$(find rotors_description)/urdf/component_snippets.xacro" />
   <link name="base_link">
@@ -24,5 +23,10 @@
     </inertial>
   </link>
-  <xacro:vi_sensor_macro namespace="${namespace}" parent_link="base_link">
+  <xacro:vi_sensor_macro
+    namespace="${namespace}"
+    parent_link="base_link"
+    enable_cameras="$(arg enable_cameras)"
+    enable_depth="$(arg enable_depth)"
+    enable_ground_truth="$(arg enable_ground_truth)">
     <origin xyz="0.0 0.0 0.6" rpy="0 0 0" />
   </xacro:vi_sensor_macro>

Commit message: added 2 new sensors, heat and rgbd camera . Also, added a new robot file for the kuri_usar package.

File: rotors_description/urdf/component_snippets.xacro (robot description, xacro)
@@ -560,5 +560,5 @@
       </collision>
       <inertial>
-        <mass value="0.170" />
+        <mass value="0.000170" />
         <origin xyz="0 0 0" />
         <inertia ixx="0.001152600" ixy="0.0" ixz="0.0"
@@ -834,5 +834,5 @@
   </xacro:macro>
   <!-- trial kinect -->
-<!--   <xacro:macro name="kinect_macro" params="namespace parent_link">
+ <!--xacro:macro name="kinect_macro" params="namespace parent_link">
   <gazebo>
 <include>
@@ -886,4 +886,5 @@
       </sensor>
 </gazebo>
-   </xacro:macro> -->
+   </xacro:macro>
+  -->
 </robot>
